Commit message: new

File: src/so100_description/urdf/so100.urdf (robot description, URDF)
Before this commit: robot so_arm100, 8 links, 7 joints
Links:
- link base: geometry collision mesh filename=package://so100_description/urdf/assets/Base.stl; visual mesh filename=package://so100_description/urdf/assets/Base.stl
- link gripper: geometry collision mesh filename=package://so100_description/urdf/assets/Fixed_Jaw.stl; visual mesh filename=package://so100_description/urdf/assets/Fixed_Jaw.stl
- link jaw: geometry collision mesh filename=package://so100_description/urdf/assets/Moving_Jaw.stl; visual mesh filename=package://so100_description/urdf/assets/Moving_Jaw.stl
- link lower_arm: geometry collision mesh filename=package://so100_description/urdf/assets/Lower_Arm.stl; visual mesh filename=package://so100_description/urdf/assets/Lower_Arm.stl
- link shoulder: geometry collision mesh filename=package://so100_description/urdf/assets/Rotation_Pitch.stl; visual mesh filename=package://so100_description/urdf/assets/Rotation_Pitch.stl
- link upper_arm: geometry collision mesh filename=package://so100_description/urdf/assets/Upper_Arm.stl; visual mesh filename=package://so100_description/urdf/assets/Upper_Arm.stl
- link wrist: geometry collision mesh filename=package://so100_description/urdf/assets/Wrist_Pitch_Roll.stl; visual mesh filename=package://so100_description/urdf/assets/Wrist_Pitch_Roll.stl
